Commit message: visualize the arm in RViz

File: urdf/Arm_Urdf.urdf (robot description, URDF)
Before this commit: robot Arm_Urdf, 18 links, 17 joints
Links:
- link Link_1: geometry collision mesh filename=package://arm_control/meshes/Link_1.STL; visual mesh filename=package://arm_control/meshes/Link_1.STL
- link Link_2: geometry collision mesh filename=package://arm_control/meshes/Link_2.STL; visual mesh filename=package://arm_control/meshes/Link_2.STL
- link Link_3: geometry collision mesh filename=package://arm_control/meshes/Link_3.STL; visual mesh filename=package://arm_control/meshes/Link_3.STL
- link Link_4: geometry collision mesh filename=package://arm_control/meshes/Link_4.STL; visual mesh filename=package://arm_control/meshes/Link_4.STL
- link Link_5: geometry collision mesh filename=package://arm_control/meshes/Link_5.STL; visual mesh filename=package://arm_control/meshes/Link_5.STL
- link Link_6: geometry collision mesh filename=package://arm_control/meshes/Link_6.STL; visual mesh filename=package://arm_control/meshes/Link_6.STL
- link base_link: geometry collision mesh filename=package://arm_control/meshes/base_link.STL; visual mesh filename=package://arm_control/meshes/base_link.STL
